Commit message: 2020/08/19

File: src/mutifingerhand_qi_urdf/urdf/gazebo_mutifingerhand_qi_urdf.urdf (robot description, URDF)
Before this commit: robot mutifingerhand, 22 links, 21 joints
Links:
- added link world
- link Plam: mass 0.1 -> 1.74090727868219
Joints:
- added joint fixed: type fixed, parent world, child Plam, origin xyz=0 0 0.25 rpy=0 0 0

File: src/mutifingerhand_qi_urdf/urdf/mutifingerhand_qi_urdf.urdf (robot description, URDF)
Before this commit: robot mutifingerhand, 22 links, 21 joints
Links:
- added link world
- link Plam: mass None -> 1.74090727868219
Joints:
- added joint virtual_joint: type fixed, parent world, child Plam, origin xyz=0 0 0.25 rpy=0 0 0
- joint J11: limit lower=-1.5 upper=0.4 effort=10 velocity=0.2 -> lower=-1.5 upper=0.4 effort=10 velocity=0.6
- joint J12: limit lower=0 upper=1.5707963267949 effort=10 velocity=0.2 -> lower=0 upper=1.5707963267949 effort=10 velocity=0.6
- joint J13: limit lower=-0.34906585039 upper=0.34906585039 effort=10 velocity=0.2 -> lower=-0.34906585039 upper=0.34906585039 effort=10 velocity=0.6
- joint J14: limit lower=0 upper=1.5707963267949 effort=10 velocity=0.2 -> lower=0 upper=1.5707963267949 effort=10 velocity=0.6
- joint J15: limit lower=0 upper=1.5707963267949 effort=10 velocity=0.2 -> lower=0 upper=1.5707963267949 effort=10 velocity=0.6
- joint J21: limit lower=0 upper=1.5707963267949 effort=10 velocity=0.2 -> lower=0 upper=1.5707963267949 effort=10 velocity=0.6
- joint J22: limit lower=-0.34906585039 upper=0.34906585039 effort=10 velocity=0.2 -> lower=-0.34906585039 upper=0.34906585039 effort=10 velocity=0.6
- joint J23: limit lower=0 upper=1.5707963267949 effort=10 velocity=0.2 -> lower=0 upper=1.5707963267949 effort=10 velocity=0.6
- joint J24: limit lower=0 upper=1.5707963267949 effort=10 velocity=0.2 -> lower=0 upper=1.5707963267949 effort=10 velocity=0.6
- joint J31: limit lower=0 upper=1.5707963267949 effort=10 velocity=0.2 -> lower=0 upper=1.5707963267949 effort=10 velocity=0.6
- joint J32: limit lower=-0.34906585039 upper=0.34906585039 effort=10 velocity=0.2 -> lower=-0.34906585039 upper=0.34906585039 effort=10 velocity=0.6
- joint J33: limit lower=0 upper=1.5707963267949 effort=10 velocity=0.2 -> lower=0 upper=1.5707963267949 effort=10 velocity=0.6
- joint J34: limit lower=0 upper=1.5707963267949 effort=10 velocity=0.2 -> lower=0 upper=1.5707963267949 effort=10 velocity=0.6
- joint J41: limit lower=0 upper=1.5707963267949 effort=10 velocity=0.2 -> lower=0 upper=1.5707963267949 effort=10 velocity=0.6
- joint J42: limit lower=-0.34906585039 upper=0.34906585039 effort=10 velocity=0.2 -> lower=-0.34906585039 upper=0.34906585039 effort=10 velocity=0.6
- joint J43: limit lower=0 upper=1.5707963267949 effort=10 velocity=0.2 -> lower=0 upper=1.5707963267949 effort=10 velocity=0.6
- joint J44: limit lower=0 upper=1.5707963267949 effort=10 velocity=0.2 -> lower=0 upper=1.5707963267949 effort=10 velocity=0.6
- joint J51: limit lower=0 upper=1.5707963267949 effort=10 velocity=0.2 -> lower=0 upper=1.5707963267949 effort=10 velocity=0.6
- joint J52: limit lower=-0.34906585039 upper=0.34906585039 effort=10 velocity=0.2 -> lower=-0.34906585039 upper=0.34906585039 effort=10 velocity=0.6
- joint J53: limit lower=0 upper=1.5707963267949 effort=10 velocity=0.2 -> lower=0 upper=1.5707963267949 effort=10 velocity=0.6
- joint J54: limit lower=0 upper=1.5707963267949 effort=10 velocity=0.2 -> lower=0 upper=1.5707963267949 effort=10 velocity=0.6
